File: stm.kicad_pcb (KiCad board)
At the start: 2 copper layers, 42 x 34 mm, 32 parts, among them J1 USB_B_Micro, J2 Conn_01x04_Pin, J3 Conn_01x04_Pin, J4 Conn_01x04_Pin, SW1 SW_SPDT, U1 AMS1117-3.3, U2 STM32F103C_8-B_Tx, Y1 16MHz

Commit message: proto
Parts:
- moved J1 0.25 mm to (153.0, 94.0)
Routing:
- net VBUS: track 0.00 -> 12.6 mm
- net +3.3V: track 152.2 -> 154.2 mm
- net /USB_D+: track 13.9 -> 12.3 mm
- removed copper zone on F.Cu, net VBUS
Changed lines of the file:
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@@
 	(footprint "Connector_USB:USB_Micro-B_Wuerth_629105150521"
 		(layer "F.Cu")
-		(at 153.245 94.025 90)
+		(at 153 94.025 90)
 		(descr "USB Micro-B receptacle, http://www.mouser.com/ds/2/445/629105150521-469306.pdf")
 		(tags "usb micro receptacle")
@@
 	)
 	(segment
+		(start 131.5875 91.4325)
+		(end 133 90.02)
+		(width 0.3)
+		(layer "F.Cu")
+		(net 1)
+	)
+	(segment
 		(start 150 110)
 		(end 141 110)
@@
 	)
 	(segment
+		(start 142.7 101.85)
+		(end 142.7 99.82)
+		(width 1)
+		(layer "F.Cu")
+		(net 4)
+	)
+	(segment
+		(start 142.7 99.82)
+		(end 145 97.52)
+		(width 1)
+		(layer "F.Cu")
+		(net 4)
+	)
+	(segment
+		(start 145 96.795)
+		(end 146.194 95.601)
+		(width 1)
+		(layer "F.Cu")
+		(net 4)
+	)
+	(segment
+		(start 145 97.52)
+		(end 145 96.795)
+		(width 1)
+		(layer "F.Cu")
+		(net 4)
+	)
+	(segment
+		(start 146.194 95.601)
+		(end 151.1 95.601)
+		(width 1)
+		(layer "F.Cu")
+		(net 4)
+	)
+	(segment
 		(start 132.499 97.503966)
 		(end 132.499 99.499)
@@
 	)
 	(segment
-		(start 151.331397 94.675)
-		(end 151.345 94.675)
-		(width 0.2)
-		(layer "F.Cu")
-		(net 10)
-	)
-	(segment
-		(start 139.9125 93.4325)
-		(end 141.018751 93.4325)
+		(start 144.856802 94.675)
+		(end 151.1 94.675)
 		(width 0.2)
 		(layer "F.Cu")
@@
 	)
 	(segment
-		(start 151.207397 94.799)
-		(end 151.331397 94.675)
+		(start 151.331397 94.675)
+		(end 151.345 94.675)
 		(width 0.2)
 		(layer "F.Cu")
@@
 	)
 	(segment
-		(start 141.018751 93.4325)
-		(end 141.043751 93.4075)
+		(start 139.9125 93.4325)
+		(end 141.018751 93.4325)
 		(width 0.2)
 		(layer "F.Cu")
@@
 	)
 	(segment
-		(start 150.394 94.799)
-		(end 151.207397 94.799)
+		(start 143.589302 93.4075)
+		(end 144.856802 94.675)
 		(width 0.2)
 		(layer "F.Cu")
@@
 	)
 	(segment
-		(start 145.406802 95.225)
-		(end 150.394 95.225)
+		(start 151.207397 94.799)
+		(end 151.331397 94.675)
 		(width 0.2)
 		(layer "F.Cu")
@@
 	)
 	(segment
-		(start 143.589302 93.4075)
-		(end 145.406802 95.225)
+		(start 141.018751 93.4325)
+		(end 141.043751 93.4075)
 		(width 0.2)
 		(layer "F.Cu")
@@
 	)
 	(segment
-		(start 150.394 95.225)
-		(end 150.394 94.799)
-		(width 0.2)
+		(start 151.1 94.675)
+		(end 150.325 94.675)
+		(width 0.3)
 		(layer "F.Cu")
 		(net 10)
 	)
 	(segment
-		(start 141.018751 92.9325)
-		(end 141.043751 92.9575)
+		(start 146.5 94.025)
+		(end 151.1 94.025)
 		(width 0.2)
 		(layer "F.Cu")
@@
 	)
 	(segment
-		(start 151.221 94.149)
-		(end 151.345 94.025)
+		(start 146.5 94.025)
+		(end 146.5 93.51)
 		(width 0.2)
 		(layer "F.Cu")
@@
 	)
 	(segment
-		(start 141.043751 92.9575)
-		(end 143.775698 92.9575)
+		(start 141.018751 92.9325)
+		(end 141.043751 92.9575)
 		(width 0.2)
 		(layer "F.Cu")
@@
 	(segment
 		(start 143.775698 92.9575)
-		(end 145.593198 94.775)
+		(end 144.843198 94.025)
 		(width 0.2)
 		(layer "F.Cu")
@@
 	)
 	(segment
-		(start 146.5 93.51)
-		(end 146.5 94.775)
-		(width 0.3)
-		(layer "F.Cu")
-		(net 14)
-	)
-	(segment
-		(start 149.94402 94.612612)
-		(end 150.407632 94.149)
+		(start 151.221 94.149)
+		(end 151.345 94.025)
 		(width 0.2)
 		(layer "F.Cu")
@@
 	)
 	(segment
-		(start 149.94402 94.775)
-		(end 149.94402 94.612612)
+		(start 141.043751 92.9575)
+		(end 143.775698 92.9575)
 		(width 0.2)
 		(layer "F.Cu")
@@
 	)
 	(segment
-		(start 145.593198 94.775)
-		(end 146.5 94.775)
+		(start 144.843198 94.025)
+		(end 146.5 94.025)
 		(width 0.2)
 		(layer "F.Cu")
@@
 	)
 	(segment
-		(start 150.407632 94.149)
-		(end 151.221 94.149)
-		(width 0.2)
-		(layer "F.Cu")
-		(net 14)
-	)
-	(segment
-		(start 146.5 94.775)
-		(end 149.94402 94.775)
-		(width 0.2)
-		(layer "F.Cu")
-		(net 14)
-	)
-	(segment
 		(start 143.5 83.5)
 		(end 143.46 83.46)
@@
 			)
 		)
-	)
-	(zone
-		(net 4)
-		(net_name "VBUS")
-		(layer "F.Cu")
-		(hatch edge 0.5)
-		(priority 3)
-		(connect_pads yes
-			(clearance 0.5)
-		)
-		(min_thickness 0.25)
-		(filled_areas_thickness no)
-		(fill yes
-			(thermal_gap 0.5)
-			(thermal_bridge_width 0.5)
-		)
-		(polygon
-			(pts
-				(xy 144 103.5) (xy 144 99.625) (xy 145.5 98.5) (xy 145.5 97) (xy 146.375 96.5625) (xy 151.5 96.05)
-				(xy 151.5 95) (xy 151 95) (xy 150.5 95.5) (xy 146 95) (xy 145 95.5) (xy 144.5 96) (xy 144 96.5)
-				(xy 144 98.5) (xy 142 99.5) (xy 141.5 100.5) (xy 141.5 103.5)
-			)
-		)
